Commit message: Fixes

File: urdf/qmini_description.urdf (robot description, URDF)
Before this commit: robot qmini_description, 12 links, 11 joints
Links:
- removed link ankle_pitch_l
- removed link ankle_pitch_r
- removed link hip_pitch_l
- removed link hip_pitch_r
- removed link hip_roll_l
- removed link hip_roll_r
- removed link hip_yaw_l
- removed link hip_yaw_r
- removed link knee_pitch_l
- removed link knee_pitch_r
- added link ankle_pitch_l_link, mass 0.44945849105282; collision mesh filename=package://qmini_description/meshes/ankle_pitch_l_link.STL; visual mesh filename=package://qmini_description/meshes/ankle_pitch_l_link.STL
- added link ankle_pitch_r_link, mass 0.449458238705845; collision mesh filename=package://qmini_description/meshes/ankle_pitch_r_link.STL; visual mesh filename=package://qmini_description/meshes/ankle_pitch_r_link.STL
- added link hip_pitch_l_link, mass 1.54138166088268; collision mesh filename=package://qmini_description/meshes/hip_pitch_l_link.STL; visual mesh filename=package://qmini_description/meshes/hip_pitch_l_link.STL
- added link hip_pitch_r_link, mass 1.54138123257867; collision mesh filename=package://qmini_description/meshes/hip_pitch_r_link.STL; visual mesh filename=package://qmini_description/meshes/hip_pitch_r_link.STL
- added link hip_roll_l_link, mass 0.144022608554608; collision mesh filename=package://qmini_description/meshes/hip_roll_l_link.STL; visual mesh filename=package://qmini_description/meshes/hip_roll_l_link.STL
- added link hip_roll_r_link, mass 0.144022449768194; collision mesh filename=package://qmini_description/meshes/hip_roll_r_link.STL; visual mesh filename=package://qmini_description/meshes/hip_roll_r_link.STL
- added link hip_yaw_l_link, mass 0.802589402885363; collision mesh filename=package://qmini_description/meshes/hip_yaw_l_link.STL; visual mesh filename=package://qmini_description/meshes/hip_yaw_l_link.STL
- added link hip_yaw_r_link, mass 0.802588717539285; collision mesh filename=package://qmini_description/meshes/hip_yaw_r_link.STL; visual mesh filename=package://qmini_description/meshes/hip_yaw_r_link.STL
- added link knee_pitch_l_link, mass 0.882230006451168; collision mesh filename=package://qmini_description/meshes/knee_pitch_l_link.STL; visual mesh filename=package://qmini_description/meshes/knee_pitch_l_link.STL
- added link knee_pitch_r_link, mass 0.882229952732639; collision mesh filename=package://qmini_description/meshes/knee_pitch_r_link.STL; visual mesh filename=package://qmini_description/meshes/knee_pitch_r_link.STL
- link base_link: mass 5.42932022155468 -> 5.90206584561033
Joints:
- joint ankle_pitch_l: child ankle_pitch_l -> ankle_pitch_l_link; origin xyz=0.0530131209926416 0.0208000020258525 -0.145652356077947 rpy=0 0 0 -> xyz=0.0530131222154821 0.0211000000000001 -0.145652356221812 rpy=0 0 0; parent knee_pitch_l -> knee_pitch_l_link
- joint ankle_pitch_r: child ankle_pitch_r -> ankle_pitch_r_link; origin xyz=0.0530131229787218 -0.020799999048718 -0.145652356080173 rpy=0 0 0 -> xyz=0.0530131222154776 -0.0207999999999969 -0.145652356221815 rpy=0 0 0; parent knee_pitch_r -> knee_pitch_r_link
- joint hip_pitch_l: child hip_pitch_l -> hip_pitch_l_link; origin xyz=-0.00149999904255326 0.0279999989589162 0 rpy=0 0 0 -> xyz=-0.0160000000000013 0.028 0 rpy=0 0 0; parent hip_roll_l -> hip_roll_l_link
- joint hip_pitch_r: child hip_pitch_r -> hip_pitch_r_link; origin xyz=-0.00150000021047648 -0.028200001941497 0 rpy=0 0 0 -> xyz=-0.0159999999999998 -0.028 0 rpy=0 0 0; parent hip_roll_r -> hip_roll_r_link
- joint hip_roll_l: child hip_roll_l -> hip_roll_l_link; origin xyz=0.0179161263785935 0.0536951934928277 -0.1073 rpy=0 0 0 -> xyz=0.0325000000000028 0.0540000000000005 -0.073 rpy=0 0 0; parent hip_yaw_l -> hip_yaw_l_link
- joint hip_roll_r: child hip_roll_r -> hip_roll_r_link; origin xyz=0.0179161246071409 -0.0536951920782032 -0.1073 rpy=0 0 0 -> xyz=0.0324999999999978 -0.0540000000000006 -0.0729999999999999 rpy=0 0 0; parent hip_yaw_r -> hip_yaw_r_link
- joint hip_yaw_l: child hip_yaw_l -> hip_yaw_l_link; origin xyz=0.0136775248726286 0.0553048691600504 -0.000799999999999912 rpy=0 0 0 -> xyz=0.0135936510211813 0.0550000626641943 -0.0350999999999998 rpy=0 0 0
- joint hip_yaw_r: child hip_yaw_r -> hip_yaw_r_link; origin xyz=0.0136775258700451 -0.0553047455885371 -0.000799999999999773 rpy=0 0 0 -> xyz=0.0135936510211862 -0.0549999373358046 -0.0350999999999998 rpy=0 0 0
- joint knee_pitch_l: child knee_pitch_l -> knee_pitch_l_link; origin xyz=-0.0813172798364506 -0.000299999426322167 -0.0813172798385736 rpy=0 0 0 -> xyz=-0.073920575113949 0 -0.0880951109586866 rpy=0 0 0; parent hip_pitch_l -> hip_pitch_l_link
- joint knee_pitch_r: child knee_pitch_r -> knee_pitch_r_link; origin xyz=-0.0813172798364519 0.000499999426317815 -0.0813172798399789 rpy=0 0 0 -> xyz=-0.0739205751139517 0 -0.0880951109586838 rpy=0 0 0; parent hip_pitch_r -> hip_pitch_r_link

Commit message: Update qmini_description.urdf

File: urdf/qmini_description.urdf (robot description, URDF)
Before this commit: robot qmini_description, 12 links, 11 joints
Joints:
- joint ankle_pitch_r: origin xyz=0.0530131222154776 -0.0207999999999969 -0.145652356221815 rpy=0 0 0 -> xyz=0.0530131222154776 -0.0211000000000001 -0.145652356221815 rpy=0 0 0
